File: phictrl/phictrl.kicad_pcb (KiCad board)
At the start: 2 copper layers, 17.7 x 15.6 mm, 10 parts, among them J1 F-RGB, J2 J-IR, J3 J-PRG, J4 J-RS232, J5 J-BT, U1 STM32F103C8Tx

Commit message: Some changes.
Parts:
- moved J1 14.2 mm to (61.5, 45.9)
- moved R1 14.2 mm to (66.1, 44.1)
- moved R2 14.2 mm to (66.2, 38.2)
- moved R3 14.2 mm to (66.3, 41.1)
- moved D1 14.2 mm to (72.8, 38.0)
Changed lines of the file:
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@@
   )
   (module LED_THT:LED_D5.0mm-4_RGB (layer F.Cu)
-    (at 85.5 44.3 270)
+    (at 72.8 37.95 270)
     (descr "LED, diameter 5.0mm, 2 pins, diameter 5.0mm, 3 pins, diameter 5.0mm, 4 pins, http://www.kingbright.com/attachments/file/psearch/000/00/00/L-154A4SUREQBFZGEW(Ver.9A).pdf")
     (tags "LED diameter 5.0mm 2 pins diameter 5.0mm 3 pins diameter 5.0mm 4 pins RGB RGBLED")
@@
   )
   (module Resistor_SMD:R_0805_2012Metric_Pad1.15x1.40mm_HandSolder (layer F.Cu)
-    (at 79 47.5)
+    (at 66.3 41.15)
     (descr "Resistor SMD 0805 (2012 Metric), square (rectangular) end terminal, IPC_7351 nominal with elongated pad for handsoldering. (Body size source: https://docs.google.com/spreadsheets/d/1BsfQQcO9C6DZCsRaXUlFlo91Tg2WpOkGARC1WS5S8t0/edit?usp=sharing), generated with kicad-footprint-generator")
     (tags "resistor handsolder")
@@
   )
   (module Resistor_SMD:R_0805_2012Metric_Pad1.15x1.40mm_HandSolder (layer F.Cu)
-    (at 78.925 44.6)
+    (at 66.225 38.25)
     (descr "Resistor SMD 0805 (2012 Metric), square (rectangular) end terminal, IPC_7351 nominal with elongated pad for handsoldering. (Body size source: https://docs.google.com/spreadsheets/d/1BsfQQcO9C6DZCsRaXUlFlo91Tg2WpOkGARC1WS5S8t0/edit?usp=sharing), generated with kicad-footprint-generator")
     (tags "resistor handsolder")
@@
   )
   (module Resistor_SMD:R_0805_2012Metric_Pad1.15x1.40mm_HandSolder (layer F.Cu)
-    (at 78.8 50.5)
+    (at 66.1 44.15)
     (descr "Resistor SMD 0805 (2012 Metric), square (rectangular) end terminal, IPC_7351 nominal with elongated pad for handsoldering. (Body size source: https://docs.google.com/spreadsheets/d/1BsfQQcO9C6DZCsRaXUlFlo91Tg2WpOkGARC1WS5S8t0/edit?usp=sharing), generated with kicad-footprint-generator")
     (tags "resistor handsolder")
@@
   )
   (module Connector_Wire:SolderWirePad_1x04_P3.81mm_Drill1mm (layer F.Cu)
-    (at 74.2 52.22 90)
+    (at 61.5 45.87 90)
     (descr "Wire solder connection")
     (tags connector)
@@
       (net 4 /led-r))
   )
-  (gr_line (start 72 54.2) (end 72 38.6) (layer Edge.Cuts) (width 0.05))
-  (gr_line (start 89.7 54.2) (end 72 54.2) (layer Edge.Cuts) (width 0.05))
-  (gr_line (start 89.7 38.6) (end 89.7 54.2) (layer Edge.Cuts) (width 0.05))
-  (gr_line (start 72 38.6) (end 89.7 38.6) (layer Edge.Cuts) (width 0.05))
-  (segment (start 77.4 41.5) (end 80.9 41.5) (width 0.7) (layer F.Cu) (net 1))
-  (segment (start 74.2 40.79) (end 76.69 40.79) (width 0.7) (layer F.Cu) (net 1))
-  (segment (start 83.7 44.3) (end 85.5 44.3) (width 0.7) (layer F.Cu) (net 1))
-  (segment (start 80.9 41.5) (end 83.7 44.3) (width 0.7) (layer F.Cu) (net 1))
-  (segment (start 76.69 40.79) (end 77.4 41.5) (width 0.7) (layer F.Cu) (net 1))
-  (segment (start 77.065 48.41) (end 77.975 47.5) (width 0.7) (layer F.Cu) (net 2))
-  (segment (start 74.2 48.41) (end 77.065 48.41) (width 0.7) (layer F.Cu) (net 2))
-  (segment (start 74.2 44.6) (end 77.9 44.6) (width 0.7) (layer F.Cu) (net 3))
-  (segment (start 76.055 52.22) (end 77.775 50.5) (width 0.7) (layer F.Cu) (net 4))
-  (segment (start 74.2 52.22) (end 76.055 52.22) (width 0.7) (layer F.Cu) (net 4))
-  (segment (start 87.5 48.8) (end 87.5 46.4) (width 0.7) (layer F.Cu) (net 5))
-  (segment (start 86.67 45.57) (end 85.5 45.57) (width 0.7) (layer F.Cu) (net 5))
-  (segment (start 87.5 46.4) (end 86.67 45.57) (width 0.7) (layer F.Cu) (net 5))
-  (segment (start 79.825 50.5) (end 85.8 50.5) (width 0.7) (layer F.Cu) (net 5))
-  (segment (start 85.8 50.5) (end 87.5 48.8) (width 0.7) (layer F.Cu) (net 5))
-  (segment (start 83.24 46.84) (end 85.5 46.84) (width 0.7) (layer F.Cu) (net 6))
-  (segment (start 79.95 44.6) (end 81 44.6) (width 0.7) (layer F.Cu) (net 6))
-  (segment (start 81 44.6) (end 83.24 46.84) (width 0.7) (layer F.Cu) (net 6))
-  (segment (start 80.635 48.11) (end 80.025 47.5) (width 0.5) (layer F.Cu) (net 7))
-  (segment (start 85.5 48.11) (end 80.635 48.11) (width 0.5) (layer F.Cu) (net 7))
+  (gr_line (start 59.3 47.85) (end 59.3 32.25) (layer Edge.Cuts) (width 0.05))
+  (gr_line (start 77 47.85) (end 59.3 47.85) (layer Edge.Cuts) (width 0.05))
+  (gr_line (start 77 32.25) (end 77 47.85) (layer Edge.Cuts) (width 0.05))
+  (gr_line (start 59.3 32.25) (end 77 32.25) (layer Edge.Cuts) (width 0.05))
+  (segment (start 64.7 35.15) (end 68.2 35.15) (width 0.7) (layer F.Cu) (net 1))
+  (segment (start 61.5 34.44) (end 63.99 34.44) (width 0.7) (layer F.Cu) (net 1))
+  (segment (start 71 37.95) (end 72.8 37.95) (width 0.7) (layer F.Cu) (net 1))
+  (segment (start 68.2 35.15) (end 71 37.95) (width 0.7) (layer F.Cu) (net 1))
+  (segment (start 63.99 34.44) (end 64.7 35.15) (width 0.7) (layer F.Cu) (net 1))
+  (segment (start 64.365 42.06) (end 65.275 41.15) (width 0.7) (layer F.Cu) (net 2))
+  (segment (start 61.5 42.06) (end 64.365 42.06) (width 0.7) (layer F.Cu) (net 2))
+  (segment (start 61.5 38.25) (end 65.2 38.25) (width 0.7) (layer F.Cu) (net 3))
+  (segment (start 63.355 45.87) (end 65.075 44.15) (width 0.7) (layer F.Cu) (net 4))
+  (segment (start 61.5 45.87) (end 63.355 45.87) (width 0.7) (layer F.Cu) (net 4))
+  (segment (start 74.8 42.45) (end 74.8 40.05) (width 0.7) (layer F.Cu) (net 5))
+  (segment (start 73.97 39.22) (end 72.8 39.22) (width 0.7) (layer F.Cu) (net 5))
+  (segment (start 74.8 40.05) (end 73.97 39.22) (width 0.7) (layer F.Cu) (net 5))
+  (segment (start 67.125 44.15) (end 73.1 44.15) (width 0.7) (layer F.Cu) (net 5))
+  (segment (start 73.1 44.15) (end 74.8 42.45) (width 0.7) (layer F.Cu) (net 5))
+  (segment (start 70.54 40.49) (end 72.8 40.49) (width 0.7) (layer F.Cu) (net 6))
+  (segment (start 67.25 38.25) (end 68.3 38.25) (width 0.7) (layer F.Cu) (net 6))
+  (segment (start 68.3 38.25) (end 70.54 40.49) (width 0.7) (layer F.Cu) (net 6))
+  (segment (start 67.935 41.76) (end 67.325 41.15) (width 0.5) (layer F.Cu) (net 7))
+  (segment (start 72.8 41.76) (end 67.935 41.76) (width 0.5) (layer F.Cu) (net 7))
 )

Commit message: Printed PCB
Parts:
- D1: value LED_CRGB -> LED_RCBG
- moved D1 5.45 mm to (70.8, 43.0), turned to 90 degrees
Connections:
- D1 pad 1: GND -> Net-(D1-Pad1)
- D1 pad 2: Net-(D1-Pad2) -> GND
- R1 pad 2: Net-(D1-Pad2) -> Net-(D1-Pad1)
- R2 pad 2: Net-(D1-Pad3) -> Net-(D1-Pad4)
- R3 pad 2: Net-(D1-Pad4) -> Net-(D1-Pad3)
Routing:
- net Net-(D1-Pad2): track 13.1 -> 0.00 mm
- net GND: track 12.8 -> 18.8 mm
- net Net-(D1-Pad1): track 0.00 -> 4.10 mm
- net Net-(D1-Pad3): track 6.48 -> 3.71 mm
- net Net-(D1-Pad4): track 5.73 -> 3.89 mm
- added copper zone on F.Cu, net GND
Other:
- board text added: "B"
- board text added: "G"
- board text added: "R"
